File: V2.kicad_pcb (KiCad board)
At the start: 2 copper layers, 430 x 118.4 mm, 264 parts, among them IC1 MCP73831-2ACI_MC, Q1 CJ2305, SW1 SW_Push, SW10 SW_Push, SW100 SW_Push, SW101 SW_Push, SW102 SW_Push, SW103 SW_Push, SW104 SW_Push, SW105 SW_Push, SW106 SW_Push, SW107 SW_Push, SW108 SW_Push, SW109 SW_Push, SW11 SW_Push, SW110 SW_Push, SW12 SW_Push, SW13 SW_Push, SW14 SW_Push, SW15 SW_Push, SW16 SW_Push, SW17 SW_Push, SW18 SW_Push, SW19 SW_Push, SW2 SW_Push, SW20 SW_Push, SW21 SW_Push, SW22 SW_Push, SW23 SW_Push, SW24 SW_Push, SW25 SW_Push, SW26 SW_Push, SW27 SW_Push, SW28 SW_Push, SW29 SW_Push, SW3 SW_Push, SW30 SW_Push, SW31 SW_Push, SW32 SW_Push, SW33 SW_Push, SW34 SW_Push, SW35 SW_Push, SW36 SW_Push, SW37 SW_Push, SW38 SW_Push, SW39 SW_Push, SW4 SW_Push, SW40 SW_Push, SW41 SW_Push, SW42 SW_Push, SW43 SW_Push, SW44 SW_Push, SW45 SW_Push, SW46 SW_Push, SW47 SW_Push, SW48 SW_Push, SW49 SW_Push, SW5 SW_Push, SW50 SW_Push, SW51 SW_Push, SW52 SW_Push, SW53 SW_Push, SW54 SW_Push, SW55 SW_Push, SW56 SW_Push, SW57 SW_Push, SW58 SW_Push, SW59 SW_Push, SW6 SW_Push, SW60 SW_Push, SW61 SW_Push, SW62 SW_Push, SW63 SW_Push, SW64 SW_Push, SW65 SW_Push, SW66 SW_Push, SW67 EC11J1525402, SW68 SW_Push, SW69 SW_Push, SW7 SW_Push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

Commit message: updated it
Parts:
- added D111: USBLC6-2SC6_C2687116, easyeda2kicad:SOT-23-6_L2.9-W1.6-P0.95-LS2.8-BL, B.Cu at (447.2, 71.0)
- C10, C9: value 8.2pF -> 6.8pF
- R4: value 1.8k -> 2k
- R6, R7: value 1M -> 200k
- moved C1 12.7 mm to (449.0, 77.2), turned to -90 degrees
- moved R5 12.7 mm to (451.6, 64.8), turned to 0 degrees
- moved D201 0.17 mm to (445.4, 68.0)
- renumbered D1000 to D201, RST_S1 to JDBG1
Connections:
- U1 pad A6: D+ -> Net-(D111-I/O1-Pad6)
- U1 pad A7: D- -> Net-(D111-I/O2-Pad4)
- U1 pad B6: D+ -> Net-(D111-I/O1-Pad6)
- U1 pad B7: D- -> Net-(D111-I/O2-Pad4)
Routing:
- net D+: track 152.4 -> 146.5 mm
- net D-: track 152.4 -> 146.4 mm
- net GND: track 184.5 -> 189.8 mm, vias 33 -> 35
- net Net-(D111-I/O2-Pad4): track 0.00 -> 4.95 mm
- net Net-(D111-I/O1-Pad6): track 0.00 -> 4.27 mm
- net +5V: track 220.2 -> 216.7 mm, vias 2 -> 0
- net Net-(IC1-STAT): track 52.5 -> 50.9 mm
- net Net-(U1-CC2): track 6.29 -> 6.10 mm, vias 0 -> 2
Other:
- board text added: "+3V3"
- board text added: "GND"
- board text added: "SWDCLK"
- board text added: "SWDIO"

Commit message: prepare for caleb aitken
Parts:
- LED1: moved to F.Cu
- moved C2 121.1 mm to (331.0, 88.5), turned to -90 degrees
- moved R1 4.16 mm to (446.6, 28.4), turned to -90 degrees
- moved U4 0.60 mm to (439.6, 43.6)
- moved LED1 0.10 mm to (445.6, 25.6)
Routing:
- net Net-(IC1-STAT): track 50.9 -> 44.3 mm
- net GND: track 189.8 -> 185.4 mm
- net VBAT: track 183.9 -> 180.5 mm
- net COL8: track 568.5 -> 565.9 mm
- net P0.04: track 169.0 -> 169.8 mm
- net Net-(LED1-K): track 2.35 -> 1.97 mm, vias 0 -> 1
- net +5V: track 216.7 -> 216.6 mm, vias 0 -> 1

Commit message: nearly ready for buying
Parts:
- SW59: footprint PCM_Switch_Keyboard_Hotswap_Kailh:SW_Hotswap_Kailh_MX_Plated_6.25u -> PCM_Switch_Keyboard_Hotswap_Kailh:SW_Hotswap_Kailh_MX_Plated
- moved C3 112.2 mm to (340.4, 102.4), turned to 90 degrees
- moved U2 107.5 mm to (343.0, 102.5), turned to -90 degrees
- moved C4 105.0 mm to (343.3, 100.0), turned to 0 degrees
- moved D96 10.9 mm to (454.9, 88.4)
- moved R2 6.60 mm to (454.0, 77.2), turned to 180 degrees
- moved C1 3.28 mm to (447.3, 74.4)
Routing:
- net +3.3V: track 165.2 -> 25.9 mm, vias 3 -> 1
- net Net-(U2-EN): track 39.1 -> 146.5 mm, vias 0 -> 2
- net SYS: track 51.0 -> 145.9 mm
- net +5V: track 216.6 -> 186.5 mm
- net GND: track 185.4 -> 172.1 mm, vias 35 -> 38
- net VBAT: track 180.5 -> 168.6 mm
- net Net-(D96-A): track 3.76 -> 9.21 mm
- net COL4: track 533.4 -> 534.9 mm, vias 9 -> 5
- net COL1: track 484.0 -> 483.2 mm, vias 8 -> 4
- net P0.04: track 169.8 -> 169.0 mm
- net COL9: track 444.1 -> 443.4 mm, vias 10 -> 8
- net COL6: track 614.6 -> 615.2 mm, vias 12 -> 6
- net COL3: track 634.8 -> 635.3 mm, vias 10 -> 6
- net COL5: track 643.3 -> 643.7 mm, vias 8 -> 4
- net COL8: track 565.9 -> 565.5 mm, vias 14 -> 6
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- added copper zone on B.Cu, net +3.3V
- added copper zone on B.Cu, net +5V
- added copper zone on B.Cu, net SYS
- added copper zone on B.Cu, net VBAT
