File: V2.kicad_pcb (KiCad board)
At the start: 2 copper layers, 430 x 118.4 mm, 265 parts, among them IC1 MCP73831-2ACI_MC, Q1 CJ2305, SW1 SW_Push, SW10 SW_Push, SW100 SW_Push, SW101 SW_Push, SW102 SW_Push, SW103 SW_Push, SW104 SW_Push, SW105 SW_Push, SW106 SW_Push, SW107 SW_Push, SW108 SW_Push, SW109 SW_Push, SW11 SW_Push, SW110 SW_Push, SW112 MST-12D18G4 SPDT SLIDE SWITCH, SW12 SW_Push, SW13 SW_Push, SW14 SW_Push, SW15 SW_Push, SW16 SW_Push, SW17 SW_Push, SW18 SW_Push, SW19 SW_Push, SW2 SW_Push, SW20 SW_Push, SW21 SW_Push, SW22 SW_Push, SW23 SW_Push, SW24 SW_Push, SW25 SW_Push, SW26 SW_Push, SW27 SW_Push, SW28 SW_Push, SW29 SW_Push, SW3 SW_Push, SW30 SW_Push, SW31 SW_Push, SW32 SW_Push, SW33 SW_Push, SW34 SW_Push, SW35 SW_Push, SW36 SW_Push, SW37 SW_Push, SW38 SW_Push, SW39 SW_Push, SW4 SW_Push, SW40 SW_Push, SW41 SW_Push, SW42 SW_Push, SW43 SW_Push, SW44 SW_Push, SW45 SW_Push, SW46 SW_Push, SW47 SW_Push, SW48 SW_Push, SW49 SW_Push, SW5 SW_Push, SW50 SW_Push, SW51 SW_Push, SW52 SW_Push, SW53 SW_Push, SW54 SW_Push, SW55 SW_Push, SW56 SW_Push, SW57 SW_Push, SW58 SW_Push, SW59 SW_Push, SW6 SW_Push, SW60 SW_Push, SW61 SW_Push, SW62 SW_Push, SW63 SW_Push, SW64 SW_Push, SW65 SW_Push, SW66 SW_Push, SW67 EC11J1525402, SW68 SW_Push, SW69 SW_Push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

Commit message: moved fucken holes
Parts:
- moved H3 3.00 mm to (32.0, 90.0)
- moved SW112 2.50 mm to (422.8, 27.2)
- moved H8 1.80 mm to (128.6, 126.8)
- moved H10 1.50 mm to (181.0, 26.1)
- moved H2 1.50 mm to (437.8, 26.1)
- moved H4 1.50 mm to (47.6, 26.1)
- moved H9 1.50 mm to (316.8, 26.1)
- moved H11 1.05 mm to (446.0, 70.0)
Routing:
- net Net-(U2-EN): track 106.2 -> 108.5 mm
- net SYS: track 140.2 -> 142.5 mm
- net COL10: track 404.1 -> 402.8 mm
Other:
- board size 430 x 118.4 mm -> 430 x 120.9 mm
Changed lines of the file:
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@@
 	(footprint "MountingHole:MountingHole_3.2mm_M3_Pad"
 		(layer "F.Cu")
-		(at 316.8 27.6)
+		(at 316.8 26.1)
 		(descr "Mounting Hole 3.2mm, M3")
 		(tags "mounting hole 3.2mm m3")
@@
 	(footprint "MountingHole:MountingHole_3.2mm_M3_Pad"
 		(layer "F.Cu")
-		(at 128.6 125)
+		(at 128.6 126.8)
 		(descr "Mounting Hole 3.2mm, M3")
 		(tags "mounting hole 3.2mm m3")
@@
 	(footprint "MountingHole:MountingHole_3.2mm_M3_Pad"
 		(layer "F.Cu")
-		(at 181 27.6)
+		(at 181 26.1)
 		(descr "Mounting Hole 3.2mm, M3")
 		(tags "mounting hole 3.2mm m3")
@@
 	(footprint "MountingHole:MountingHole_3.2mm_M3_Pad"
 		(layer "F.Cu")
-		(at 446 68.95)
+		(at 446 70)
 		(descr "Mounting Hole 3.2mm, M3")
 		(tags "mounting hole 3.2mm m3")
@@
 	(footprint "MountingHole:MountingHole_3.2mm_M3_Pad"
 		(layer "F.Cu")
-		(at 47.6 27.6)
+		(at 47.6 26.1)
 		(descr "Mounting Hole 3.2mm, M3")
 		(tags "mounting hole 3.2mm m3")
@@
 	(footprint "MountingHole:MountingHole_3.2mm_M3_Pad"
 		(layer "F.Cu")
-		(at 32 87)
+		(at 32 90)
 		(descr "Mounting Hole 3.2mm, M3")
 		(tags "mounting hole 3.2mm m3")
@@
 	(footprint "MountingHole:MountingHole_3.2mm_M3_Pad"
 		(layer "F.Cu")
-		(at 437.8 27.6)
+		(at 437.8 26.1)
 		(descr "Mounting Hole 3.2mm, M3")
 		(tags "mounting hole 3.2mm m3")
@@
 	(footprint "easyeda2kicad:SW-SMD_MST-12D18G4-SPDT-SLIDE-SWITCH"
 		(layer "F.Cu")
-		(at 424.8 28.7 180)
+		(at 422.8 27.2 180)
 		(property "Reference" "SW112"
 			(at 0 -4 0)
@@
 	)
 	(gr_line
-		(start 28 27)
+		(start 28 24.5)
 		(end 28 64.59133)
 		(stroke
@@
 	)
 	(gr_arc
-		(start 28 27)
-		(mid 28.997912 24.599633)
-		(end 31.4 23.6)
+		(start 28 24.5)
+		(mid 28.998773 22.098773)
+		(end 31.4 21.1)
 		(stroke
 			(width 0.05)
@@
 	)
 	(gr_line
-		(start 454.6 23.6)
-		(end 31.4 23.6)
+		(start 454.6 21.1)
+		(end 31.4 21.1)
 		(stroke
 			(width 0.05)
@@
 	)
 	(gr_arc
-		(start 454.6 23.6)
-		(mid 457.002077 24.596191)
-		(end 458 27)
+		(start 454.6 21.1)
+		(mid 457.002077 22.096191)
+		(end 458 24.5)
 		(stroke
 			(width 0.05)
@@
 	)
 	(gr_line
-		(start 458 27)
+		(start 458 24.5)
 		(end 458 64.48737)
 		(stroke
@@
 	)
 	(segment
-		(start 427.3 32.2)
-		(end 427.3 28.7)
+		(start 425.3 27.2)
+		(end 427.3 29.2)
+		(width 0.2)
+		(layer "F.Cu")
+		(net "SYS")
+	)
+	(segment
+		(start 427.3 29.2)
+		(end 427.3 32.2)
 		(width 0.2)
 		(layer "F.Cu")
@@
 	)
 	(segment
-		(start 424.8 28.7)
-		(end 424.8 31)
+		(start 379.6 69.2)
+		(end 379.6 72.2)
 		(width 0.2)
 		(layer "F.Cu")
@@
 	)
 	(segment
-		(start 379.6 69.2)
-		(end 379.6 72.2)
+		(start 424.8 31)
+		(end 424.8 29.2)
+		(width 0.2)
+		(layer "F.Cu")
+		(net "Net-(U2-EN)")
+	)
+	(segment
+		(start 424.8 29.2)
+		(end 422.8 27.2)
 		(width 0.2)
 		(layer "F.Cu")
@@
 	)
 	(segment
-		(start 320 29.8)
-		(end 318.4 31.4)
-		(width 0.2)
-		(layer "F.Cu")
-		(net "COL10")
-	)
-	(segment
 		(start 398.395 86.4)
 		(end 379.5 86.4)
@@
 	)
 	(segment
-		(start 315 31.4)
-		(end 313.500001 29.900001)
-		(width 0.2)
-		(layer "F.Cu")
-		(net "COL10")
-	)
-	(segment
-		(start 398.4 101)
-		(end 398.4 96.2)
+		(start 320 29.8)
+		(end 319.899999 29.900001)
 		(width 0.2)
 		(layer "F.Cu")
@@
 	)
 	(segment
-		(start 313.500001 29.900001)
+		(start 319.899999 29.900001)
 		(end 239.6 29.900001)
 		(width 0.2)
@@
 	)
 	(segment
-		(start 399.145 55.21)
-		(end 399.145 66.2)
+		(start 398.4 101)
+		(end 398.4 96.2)
 		(width 0.2)
 		(layer "F.Cu")
@@
 	)
 	(segment
-		(start 318.4 31.4)
-		(end 315 31.4)
+		(start 399.145 55.21)
+		(end 399.145 66.2)
 		(width 0.2)
 		(layer "F.Cu")
