File: power.kicad_sch (KiCad schematic)
At the start: 17 parts, among them IC1 MCP73831-2ACI_MC, Q1 CJ2305, U1 MC-121-L124, U2 TPS7A0233DBVR, U4 S2B-PH-K-S

Commit message: updated it
Parts:
- added D111: USBLC6-2SC6_C2687116, easyeda2kicad:SOT-23-6_L2.9-W1.6-P0.95-LS2.8-BL, symbol easyeda2kicad:USBLC6-2SC6_C2687116
- R4: value 1.8k -> 2k; LCSC Part C4177 -> C22975
- renumbered D1000 to D201
Connections:
- net +5V: now also D111.5 (VBUS)
- net D+: now also D111.1 (I/O1); no longer U1.A6 (D+), U1.B6 (D+)
- net D-: now also D111.3 (I/O2); no longer U1.A7 (D-), U1.B7 (D-)
- net GND: now also D111.2 (GND)
- new net: D111.4 (I/O2), U1.A7 (D-), U1.B7 (D-)
- new net: D111.6 (I/O1), U1.A6 (D+), U1.B6 (D+)

Commit message: prepare for caleb aitken
Other:
- moved on the sheet: C2, U4
Changed lines of the file:
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@@
-	)
-	(junction
-		(at 64.77 83.82)
-		(diameter 0)
-		(color 0 0 0 0)
 	)
 	(junction
@@
 	)
 	(junction
-		(at 173.99 104.14)
+		(at 182.88 104.14)
 		(diameter 0)
 		(color 0 0 0 0)
@@
 	)
 	(junction
-		(at 173.99 102.87)
-		(diameter 0)
-		(color 0 0 0 0)
-	)
-	(junction
-		(at 154.94 104.14)
+		(at 139.7 120.65)
+		(diameter 0)
+		(color 0 0 0 0)
+	)
+	(junction
+		(at 182.88 102.87)
+		(diameter 0)
+		(color 0 0 0 0)
+	)
+	(junction
+		(at 163.83 104.14)
 		(diameter 0)
 		(color 0 0 0 0)
@@
 	)
 	(junction
-		(at 160.02 120.65)
+		(at 168.91 120.65)
 		(diameter 0)
 		(color 0 0 0 0)
@@
 	)
 	(junction
-		(at 160.02 104.14)
+		(at 168.91 104.14)
 		(diameter 0)
 		(color 0 0 0 0)
@@
 	)
 	(junction
-		(at 154.94 120.65)
+		(at 163.83 120.65)
 		(diameter 0)
 		(color 0 0 0 0)
@@
 	(junction
 		(at 257.81 114.3)
-		(diameter 0)
-		(color 0 0 0 0)
-	)
-	(junction
-		(at 139.7 120.65)
 		(diameter 0)
 		(color 0 0 0 0)
@@
 	(wire
 		(pts
-			(xy 160.02 104.14) (xy 173.99 104.14)
+			(xy 168.91 104.14) (xy 182.88 104.14)
 		)
 		(stroke
@@
 	(wire
 		(pts
-			(xy 154.94 120.65) (xy 160.02 120.65)
+			(xy 163.83 120.65) (xy 168.91 120.65)
 		)
 		(stroke
@@
 	(wire
 		(pts
-			(xy 154.94 114.3) (xy 154.94 120.65)
+			(xy 163.83 114.3) (xy 163.83 120.65)
 		)
 		(stroke
@@
 	(wire
 		(pts
-			(xy 64.77 83.82) (xy 87.63 83.82)
-		)
-		(stroke
-			(width 0)
-			(type default)
-		)
-	)
-	(wire
-		(pts
 			(xy 267.97 120.65) (xy 257.81 120.65)
 		)
@@
 	(wire
 		(pts
-			(xy 154.94 104.14) (xy 154.94 106.68)
+			(xy 163.83 104.14) (xy 163.83 106.68)
 		)
 		(stroke
@@
 	(wire
 		(pts
-			(xy 173.99 102.87) (xy 173.99 104.14)
+			(xy 182.88 102.87) (xy 182.88 104.14)
 		)
 		(stroke
@@
 	(wire
 		(pts
-			(xy 173.99 104.14) (xy 220.98 104.14)
+			(xy 182.88 104.14) (xy 220.98 104.14)
 		)
 		(stroke
@@
 	(wire
 		(pts
-			(xy 160.02 104.14) (xy 160.02 109.22)
+			(xy 168.91 104.14) (xy 168.91 109.22)
 		)
 		(stroke
@@
 	(wire
 		(pts
-			(xy 160.02 111.76) (xy 160.02 120.65)
+			(xy 168.91 111.76) (xy 168.91 120.65)
 		)
 		(stroke
@@
 	(wire
 		(pts
-			(xy 160.02 120.65) (xy 198.12 120.65)
+			(xy 168.91 120.65) (xy 198.12 120.65)
 		)
 		(stroke
@@
 	(wire
 		(pts
-			(xy 173.99 100.33) (xy 173.99 102.87)
-		)
-		(stroke
-			(width 0)
-			(type default)
-		)
-	)
-	(wire
-		(pts
-			(xy 170.18 102.87) (xy 173.99 102.87)
+			(xy 182.88 100.33) (xy 182.88 102.87)
+		)
+		(stroke
+			(width 0)
+			(type default)
+		)
+	)
+	(wire
+		(pts
+			(xy 179.07 102.87) (xy 182.88 102.87)
 		)
 		(stroke
@@
 	(wire
 		(pts
-			(xy 133.35 104.14) (xy 154.94 104.14)
+			(xy 133.35 104.14) (xy 163.83 104.14)
 		)
 		(stroke
@@
 	(wire
 		(pts
-			(xy 154.94 104.14) (xy 160.02 104.14)
-		)
-		(stroke
-			(width 0)
-			(type default)
-		)
-	)
-	(wire
-		(pts
-			(xy 139.7 120.65) (xy 154.94 120.65)
+			(xy 163.83 104.14) (xy 168.91 104.14)
+		)
+		(stroke
+			(width 0)
+			(type default)
+		)
+	)
+	(wire
+		(pts
+			(xy 139.7 120.65) (xy 163.83 120.65)
 		)
 		(stroke
@@
 	(global_label "VBAT"
 		(shape input)
-		(at 173.99 100.33 0)
+		(at 182.88 100.33 0)
 		(fields_autoplaced yes)
 		(effects
@@
 		)
 		(property "Intersheetrefs" "${INTERSHEET_REFS}"
-			(at 181.39 100.33 0)
+			(at 190.28 100.33 0)
 			(hide yes)
 			(show_name no)
@@
 	(symbol
 		(lib_id "power:PWR_FLAG")
-		(at 170.18 102.87 0)
+		(at 179.07 102.87 0)
 		(unit 1)
 		(body_style 1)
@@
 		(fields_autoplaced yes)
 		(property "Reference" "#FLG03"
-			(at 170.18 100.965 0)
+			(at 179.07 100.965 0)
 			(hide yes)
 			(show_name no)
@@
 		)
 		(property "Value" "PWR_FLAG"
-			(at 170.18 97.79 0)
+			(at 179.07 97.79 0)
 			(show_name no)
 			(do_not_autoplace no)
@@
 		)
 		(property "Footprint" ""
-			(at 170.18 102.87 0)
+			(at 179.07 102.87 0)
 			(hide yes)
 			(show_name no)
@@
 		)
 		(property "Datasheet" ""
-			(at 170.18 102.87 0)
+			(at 179.07 102.87 0)
 			(hide yes)
 			(show_name no)
@@
 		)
 		(property "Description" "Special symbol for telling ERC where power comes from"
-			(at 170.18 102.87 0)
+			(at 179.07 102.87 0)
 			(hide yes)
 			(show_name no)
@@
 	(symbol
 		(lib_id "Device:C")
-		(at 154.94 110.49 0)
+		(at 163.83 110.49 0)
 		(unit 1)
 		(body_style 1)
@@
 		(dnp no)
 		(property "Reference" "C2"
-			(at 148.082 108.966 0)
+			(at 156.972 108.966 0)
 			(show_name no)
 			(do_not_autoplace no)
@@
 		)
 		(property "Value" "4.7uF"
-			(at 146.812 111.506 0)
+			(at 155.702 111.506 0)
 			(show_name no)
 			(do_not_autoplace no)
@@
 		)
 		(property "Footprint" "Capacitor_SMD:C_0603_1608Metric"
-			(at 155.9052 114.3 0)
+			(at 164.7952 114.3 0)
 			(hide yes)
 			(show_name no)
@@
 		)
 		(property "Datasheet" ""
-			(at 154.94 110.49 0)
+			(at 163.83 110.49 0)
 			(hide yes)
 			(show_name no)
@@
 		)
 		(property "Description" "Unpolarized capacitor"
-			(at 154.94 110.49 0)
+			(at 163.83 110.49 0)
 			(hide yes)
 			(show_name no)
@@
 		)
 		(property "LCSC Part" "C19666"
-			(at 154.94 110.49 0)
+			(at 163.83 110.49 0)
 			(hide yes)
 			(show_name no)
@@
 	(symbol
 		(lib_id "easyeda2kicad:S2B-PH-K-S")
-		(at 165.1 110.49 0)
+		(at 173.99 110.49 0)
 		(unit 1)
 		(body_style 1)
@@
 		(fields_autoplaced yes)
 		(property "Reference" "U4"
-			(at 171.45 109.2199 0)
+			(at 180.34 109.2199 0)
 			(show_name no)
 			(do_not_autoplace no)
@@
 		)
 		(property "Value" "S2B-PH-K-S"
-			(at 171.45 111.7599 0)
+			(at 180.34 111.7599 0)
 			(show_name no)
 			(do_not_autoplace no)
@@
 		)
 		(property "Footprint" "easyeda2kicad:CONN-TH_S2B-PH-K-S-LF-SN"
-			(at 165.1 119.38 0)
+			(at 173.99 119.38 0)
 			(hide yes)
 			(show_name no)
@@
 		)
 		(property "Datasheet" "https://lcsc.com/product-detail/PH-Connectors_JST-Sales-America_S2B-PH-K-S-LF-SN_JST-Sales-America-S2B-PH-K-S-LF-SN_C173752.html"
-			(at 165.1 121.92 0)
+			(at 173.99 121.92 0)
 			(hide yes)
 			(show_name no)
@@
 		)
 		(property "Description" ""
-			(at 165.1 110.49 0)
+			(at 173.99 110.49 0)
 			(hide yes)
 			(show_name no)
@@
 		)
 		(property "Manufacturer" "JST"
-			(at 165.1 124.46 0)
+			(at 173.99 124.46 0)
 			(hide yes)
 			(show_name no)
@@
 		)
 		(property "MPN" "S2B-PH-K-S(LF)(SN)"
-			(at 165.1 127 0)
+			(at 173.99 127 0)
 			(hide yes)
 			(show_name no)
@@
 		)
 		(property "LCSC Part" "C173752"
-			(at 165.1 129.54 0)
-			(hide yes)
-			(show_name no)
+			(at 173.99 129.54 0)
+			(hide yes)
+			(show_name no)

Commit message: v2.3 board ;(
Parts:
- removed PWR_S1: MSK12C02, easyeda2kicad:SW-TH_MSK12C02, symbol easyeda2kicad:MSK12C02
- added SW112: MST-12D18G4 SPDT SLIDE SWITCH, easyeda2kicad:SW-SMD_MST-12D18G4-SPDT-SLIDE-SWITCH, symbol easyeda2kicad:MST-12D18G4SPDTSLIDESWITCH
Connections:
- net GND: now also SW112.3
- net SYS: now also SW112.1
- net at U2.3 (EN): now also SW112.2
Changed lines of the file:
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@@
 	)
 	(junction
-		(at 257.81 100.33)
-		(diameter 0)
-		(color 0 0 0 0)
-	)
-	(junction
 		(at 229.87 109.22)
 		(diameter 0)
@@
 	(wire
 		(pts
-			(xy 247.65 52.07) (xy 247.65 50.8)
-		)
-		(stroke
-			(width 0)
-			(type default)
-		)
-	)
-	(wire
-		(pts
 			(xy 198.12 78.74) (xy 213.36 78.74)
 		)
@@
 	(wire
 		(pts
-			(xy 250.19 100.33) (xy 257.81 100.33)
+			(xy 252.73 100.33) (xy 257.81 100.33)
 		)
 		(stroke
@@
 	(wire
 		(pts
+			(xy 252.73 50.8) (xy 252.73 100.33)
+		)
+		(stroke
+			(width 0)
+			(type default)
+		)
+	)
+	(wire
+		(pts
 			(xy 92.71 60.96) (xy 96.52 60.96)
 		)
@@
 	(wire
 		(pts
-			(xy 233.68 52.07) (xy 247.65 52.07)
+			(xy 233.68 68.58) (xy 247.65 68.58)
 		)
 		(stroke
@@
 	(wire
 		(pts
-			(xy 233.68 52.07) (xy 233.68 114.3)
+			(xy 233.68 68.58) (xy 233.68 114.3)
 		)
 		(stroke
@@
 	(wire
 		(pts
-			(xy 257.81 43.18) (xy 257.81 100.33)
+			(xy 267.97 104.14) (xy 271.78 104.14)
 		)
 		(stroke
@@
 	(wire
 		(pts
-			(xy 267.97 104.14) (xy 271.78 104.14)
+			(xy 33.02 120.65) (xy 34.29 120.65)
 		)
 		(stroke
@@
 	(wire
 		(pts
-			(xy 33.02 120.65) (xy 34.29 120.65)
+			(xy 163.83 104.14) (xy 168.91 104.14)
 		)
 		(stroke
@@
 	(wire
 		(pts
-			(xy 163.83 104.14) (xy 168.91 104.14)
+			(xy 247.65 50.8) (xy 247.65 68.58)
 		)
 		(stroke
@@
 	(wire
 		(pts
-			(xy 240.03 50.8) (xy 229.87 50.8)
+			(xy 229.87 50.8) (xy 242.57 50.8)
 		)
 		(stroke
@@
 		)
 	)
-	(wire
-		(pts
-			(xy 250.19 50.8) (xy 250.19 100.33)
-		)
-		(stroke
-			(width 0)
-			(type default)
-		)
-	)
 	(global_label "VBAT"
 		(shape input)
@@
 		)
 		(instances
-			(project "V2"
+			(project "V2.3"
 				(path "/85bcdc0c-8dc1-43cb-ba77-3dcf7ad94591/d7d5c39e-2bba-40e3-928a-00399b022351"
 					(reference "R3")
@@
 		)
 		(instances
-			(project "V2"
+			(project "V2.3"
 				(path "/85bcdc0c-8dc1-43cb-ba77-3dcf7ad94591/d7d5c39e-2bba-40e3-928a-00399b022351"
 					(reference "#PWR03")
@@
 		)
 		(instances
-			(project "V2"
+			(project "V2.3"
 				(path "/85bcdc0c-8dc1-43cb-ba77-3dcf7ad94591/d7d5c39e-2bba-40e3-928a-00399b022351"
 					(reference "D201")
@@
 		)
 		(instances
-			(project "V2"
+			(project "V2.3"
 				(path "/85bcdc0c-8dc1-43cb-ba77-3dcf7ad94591/d7d5c39e-2bba-40e3-928a-00399b022351"
 					(reference "LED1")
@@
 		)
 		(instances
-			(project "V2"
+			(project "V2.3"
 				(path "/85bcdc0c-8dc1-43cb-ba77-3dcf7ad94591/d7d5c39e-2bba-40e3-928a-00399b022351"
 					(reference "R1")
@@
 		)
 		(instances
-			(project "V2"
+			(project "V2.3"
 				(path "/85bcdc0c-8dc1-43cb-ba77-3dcf7ad94591/d7d5c39e-2bba-40e3-928a-00399b022351"
 					(reference "#FLG03")
@@
 		)
 		(instances
-			(project "V2"
+			(project "V2.3"
 				(path "/85bcdc0c-8dc1-43cb-ba77-3dcf7ad94591/d7d5c39e-2bba-40e3-928a-00399b022351"
 					(reference "C2")
@@
 		)
 		(instances
-			(project "V2"
+			(project "V2.3"
 				(path "/85bcdc0c-8dc1-43cb-ba77-3dcf7ad94591/d7d5c39e-2bba-40e3-928a-00399b022351"
 					(reference "Q1")
@@
 		)
 		(instances
-			(project "V2"
+			(project "V2.3"
 				(path "/85bcdc0c-8dc1-43cb-ba77-3dcf7ad94591/d7d5c39e-2bba-40e3-928a-00399b022351"
 					(reference "#PWR02")
@@
 		)
 		(instances
-			(project "V2"
+			(project "V2.3"
 				(path "/85bcdc0c-8dc1-43cb-ba77-3dcf7ad94591/d7d5c39e-2bba-40e3-928a-00399b022351"
 					(reference "IC1")
@@
 		)
 		(instances
-			(project "V2"
+			(project "V2.3"
 				(path "/85bcdc0c-8dc1-43cb-ba77-3dcf7ad94591/d7d5c39e-2bba-40e3-928a-00399b022351"
 					(reference "U2")
@@
 		)
 		(instances
-			(project "V2"
+			(project "V2.3"
 				(path "/85bcdc0c-8dc1-43cb-ba77-3dcf7ad94591/d7d5c39e-2bba-40e3-928a-00399b022351"
 					(reference "#FLG01")
@@
 		)
 		(instances
-			(project "V2"
+			(project "V2.3"
 				(path "/85bcdc0c-8dc1-43cb-ba77-3dcf7ad94591/d7d5c39e-2bba-40e3-928a-00399b022351"
 					(reference "U4")
@@
 		)
 		(instances
-			(project "V2"
+			(project "V2.3"
 				(path "/85bcdc0c-8dc1-43cb-ba77-3dcf7ad94591/d7d5c39e-2bba-40e3-928a-00399b022351"
 					(reference "C4")
@@
 		)
 		(instances
-			(project "V2"
+			(project "V2.3"
 				(path "/85bcdc0c-8dc1-43cb-ba77-3dcf7ad94591/d7d5c39e-2bba-40e3-928a-00399b022351"
 					(reference "R4")
@@
 	)
 	(symbol
-		(lib_id "easyeda2kicad:MSK12C02")
-		(at 247.65 44.45 0)
-		(mirror x)
+		(lib_id "easyeda2kicad:MST-12D18G4SPDTSLIDESWITCH")
+		(at 246.38 48.26 0)
 		(unit 1)
 		(body_style 1)
@@
 		(in_pos_files yes)
 		(dnp no)
-		(property "Reference" "PWR_S1"
-			(at 246.3801 36.83 90)
+		(fields_autoplaced yes)
+		(property "Reference" "SW112"
+			(at 247.65 40.64 0)
 			(show_name no)
 			(do_not_autoplace no)
@@
 					(size 1.27 1.27)
 				)
-				(justify right)
 			)
 		)
-		(property "Value" "MSK12C02"
-			(at 243.8401 36.83 90)
+		(property "Value" "MST-12D18G4 SPDT SLIDE SWITCH"
+			(at 247.65 43.18 0)
 			(show_name no)
 			(do_not_autoplace no)
@@
 					(size 1.27 1.27)
 				)
-				(justify right)
 			)
 		)
-		(property "Footprint" "easyeda2kicad:SW-TH_MSK12C02"
-			(at 247.65 35.56 0)
+		(property "Footprint" "easyeda2kicad:SW-SMD_MST-12D18G4-SPDT-SLIDE-SWITCH"
+			(at 246.38 58.42 0)
 			(hide yes)
 			(show_name no)
@@
 			)
 		)
-		(property "Datasheet" "https://lcsc.com/product-detail/Toggle-Switches_SHOU-HAN-MSK12C02_C431540.html"
-			(at 247.65 33.02 0)
+		(property "Datasheet" "https://www.lcsc.com/datasheet/C49023767.pdf"
+			(at 246.38 60.96 0)
 			(hide yes)
 			(show_name no)
@@
 		)
 		(property "Description" ""
-			(at 247.65 44.45 0)
+			(at 246.38 48.26 0)
 			(hide yes)
 			(show_name no)
@@
 		)
 		(property "Manufacturer" "SHOU HAN(首韩)"
-			(at 247.65 30.48 0)
+			(at 246.38 63.5 0)
 			(hide yes)
 			(show_name no)
@@
 			)
 		)
-		(property "MPN" "MSK12C02"
-			(at 247.65 27.94 0)
+		(property "MPN" "MST-12D18G4 SPDT Slide Switch"
+			(at 246.38 66.04 0)
 			(hide yes)
 			(show_name no)
@@
 			)
 		)
-		(property "LCSC Part" "C431540"
-			(at 247.65 25.4 0)
+		(property "LCSC Part" "C49023767"
+			(at 246.38 68.58 0)
 			(hide yes)
 			(show_name no)
@@
 			)
 		)
-		(pin "2"
+		(pin "3"
 		)
 		(pin "1"
 		)
-		(pin "4"
-		)
-		(pin "3"
+		(pin "2"
 		)
 		(instances
-			(project "V2"
+			(project "V2.3"
 				(path "/85bcdc0c-8dc1-43cb-ba77-3dcf7ad94591/d7d5c39e-2bba-40e3-928a-00399b022351"
-					(reference "PWR_S1")
+					(reference "SW112")
 					(unit 1)
 				)
@@
 		)
 		(instances
-			(project "V2"
+			(project "V2.3"
 				(path "/85bcdc0c-8dc1-43cb-ba77-3dcf7ad94591/d7d5c39e-2bba-40e3-928a-00399b022351"
 					(reference "C1")
@@
 		)
 		(instances
-			(project "V2"
+			(project "V2.3"
 				(path "/85bcdc0c-8dc1-43cb-ba77-3dcf7ad94591/d7d5c39e-2bba-40e3-928a-00399b022351"
 					(reference "D111")
@@
 		)
 		(instances
-			(project "V2"
+			(project "V2.3"
 				(path "/85bcdc0c-8dc1-43cb-ba77-3dcf7ad94591/d7d5c39e-2bba-40e3-928a-00399b022351"
 					(reference "R5")
@@
 		)
 		(instances
-			(project "V2"
+			(project "V2.3"
 				(path "/85bcdc0c-8dc1-43cb-ba77-3dcf7ad94591/d7d5c39e-2bba-40e3-928a-00399b022351"
 					(reference "#FLG02")
@@
 		)
 		(instances
-			(project "V2"
+			(project "V2.3"
 				(path "/85bcdc0c-8dc1-43cb-ba77-3dcf7ad94591/d7d5c39e-2bba-40e3-928a-00399b022351"
 					(reference "U1")
@@
 		)
 		(instances
-			(project "V2"
+			(project "V2.3"
 				(path "/85bcdc0c-8dc1-43cb-ba77-3dcf7ad94591/d7d5c39e-2bba-40e3-928a-00399b022351"
 					(reference "#PWR01")
@@
 		)
 		(instances
-			(project "V2"
+			(project "V2.3"
 				(path "/85bcdc0c-8dc1-43cb-ba77-3dcf7ad94591/d7d5c39e-2bba-40e3-928a-00399b022351"
 					(reference "R2")
@@
 		)
 		(instances
-			(project "V2"
+			(project "V2.3"
 				(path "/85bcdc0c-8dc1-43cb-ba77-3dcf7ad94591/d7d5c39e-2bba-40e3-928a-00399b022351"
 					(reference "C3")
@@
 		)
 		(instances
-			(project "V2"
+			(project "V2.3"
 				(path "/85bcdc0c-8dc1-43cb-ba77-3dcf7ad94591/d7d5c39e-2bba-40e3-928a-00399b022351"
 					(reference "#FLG04")
